File: robot_pocketbeagle_pcb/robot_pocketbeagle.kicad_sch (KiCad schematic)
At the start: 104 parts, among them J1 QMC5883L, J10 driver_dvr8833, J12 IN_DVR8833, J13 9V_DC_DC, J14 servo_x_y, J15 shr05, J16 5V_DC_DC, J17 Conn_GND, J18 Conn_5V, J19 Conn_pwm_out_b, J2 USB_A, J20 Conn_pwm_out_a, J21 Conn_P2_3.3V, J29 Conn_AIN_4.096_3.3_1.8V, J3 UART0, J30 Conn_5V, J31 Conn_GPI028_34, J4 P1, J5 MPU6050, J6 ADS1115, J7 P2, J8 Conn_i2c2, J9 OUT_DVR8833, Q1 BC847, Q2 BC847, Q3 QM6015D, Q4 BC847, Q5 BC847, Q6 QM6015D, Q7 QM6015D, U1 PC817, U2 PC817, U3 74HC00, U4 LM358, U5 L7805_REZERV

Commit message: add doc and fix shem board
Parts:
- C5: value 33n -> 330n
- C6: value 1n -> 100n
- R1, R2: value 1K -> 180
- R14: value 150K -> 1.5K
- R15: value 75K -> 750
- R16: value 430K -> 4.3K
- R17: value 100K -> 1K
- R18: value 110K -> 2k
- R21: value 100K -> 1.5k
- R30: value 110K -> 2K
- R31: value 100K -> 1.5K
- R41: value 2K -> 350
- R8: value 3K -> 3.3K
Changed lines of the file:
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@@
       (effects (font (size 1.27 1.27)) (justify left))
     )
-    (property "Value" "33n" (id 1) (at 247.65 160.0199 0)
+    (property "Value" "330n" (id 1) (at 247.65 160.0199 0)
       (effects (font (size 1.27 1.27)) (justify left))
     )
@@
       (effects (font (size 1.27 1.27)) (justify left))
     )
-    (property "Value" "110K" (id 1) (at 274.32 229.8699 0)
+    (property "Value" "2K" (id 1) (at 274.32 229.8699 0)
       (effects (font (size 1.27 1.27)) (justify left))
     )
@@
       (effects (font (size 1.27 1.27)) (justify left))
     )
-    (property "Value" "75K" (id 1) (at 83.82 194.3101 0)
+    (property "Value" "750" (id 1) (at 83.82 194.3101 0)
       (effects (font (size 1.27 1.27)) (justify left))
     )
@@
       (effects (font (size 1.27 1.27)) (justify left))
     )
-    (property "Value" "1n" (id 1) (at 274.32 160.0199 0)
+    (property "Value" "100n" (id 1) (at 274.32 160.0199 0)
       (effects (font (size 1.27 1.27)) (justify left))
     )
@@
       (effects (font (size 1.27 1.27)) (justify left))
     )
-    (property "Value" "110K" (id 1) (at 274.32 193.0399 0)
+    (property "Value" "2k" (id 1) (at 274.32 193.0399 0)
       (effects (font (size 1.27 1.27)) (justify left))
     )
@@
   (symbol (lib_id "Device:R") (at 220.98 52.07 90) (unit 1)
     (in_bom yes) (on_board yes) (fields_autoplaced)
-    (property "Reference" "R1" (id 0) (at 219.7099 49.53 0)
-      (effects (font (size 1.27 1.27)) (justify left))
-    )
-    (property "Value" "1K" (id 1) (at 222.2499 49.53 0)
-      (effects (font (size 1.27 1.27)) (justify left))
-    )
+    (property "Reference" "R1" (id 0) (at 220.98 45.72 90))
+    (property "Value" "180" (id 1) (at 220.98 48.26 90))
     (property "Footprint" "Resistor_SMD:R_0805_2012Metric" (id 2) (at 220.98 53.848 90)
       (effects (font (size 1.27 1.27)) hide)
@@
       (effects (font (size 1.27 1.27)) (justify left))
     )
-    (property "Value" "150K" (id 1) (at 83.82 184.1501 0)
+    (property "Value" "1.5K" (id 1) (at 83.82 184.1501 0)
       (effects (font (size 1.27 1.27)) (justify left))
     )
@@
       (effects (font (size 1.27 1.27)) (justify left))
     )
-    (property "Value" "430K" (id 1) (at 83.82 208.2801 0)
+    (property "Value" "4.3K" (id 1) (at 83.82 208.2801 0)
       (effects (font (size 1.27 1.27)) (justify left))
     )
@@
   (symbol (lib_id "Device:R") (at 220.98 68.58 90) (unit 1)
     (in_bom yes) (on_board yes) (fields_autoplaced)
-    (property "Reference" "R2" (id 0) (at 219.7099 66.04 0)
-      (effects (font (size 1.27 1.27)) (justify left))
-    )
-    (property "Value" "1K" (id 1) (at 222.2499 66.04 0)
-      (effects (font (size 1.27 1.27)) (justify left))
-    )
+    (property "Reference" "R2" (id 0) (at 220.98 62.23 90))
+    (property "Value" "180" (id 1) (at 220.98 64.77 90))
     (property "Footprint" "Resistor_SMD:R_0805_2012Metric" (id 2) (at 220.98 70.358 90)
       (effects (font (size 1.27 1.27)) hide)
@@
       (effects (font (size 1.27 1.27)) (justify left))
     )
-    (property "Value" "100K" (id 1) (at 83.82 218.4401 0)
+    (property "Value" "1K" (id 1) (at 83.82 218.4401 0)
       (effects (font (size 1.27 1.27)) (justify left))
     )
@@
       (effects (font (size 1.27 1.27)) (justify left))
     )
-    (property "Value" "2K" (id 1) (at 245.1101 118.11 0)
+    (property "Value" "350" (id 1) (at 245.1101 118.11 0)
       (effects (font (size 1.27 1.27)) (justify left))
     )
@@
       (effects (font (size 1.27 1.27)) (justify left))
     )
-    (property "Value" "100K" (id 1) (at 274.32 237.4899 0)
+    (property "Value" "1.5K" (id 1) (at 274.32 237.4899 0)
       (effects (font (size 1.27 1.27)) (justify left))
     )
@@
       (effects (font (size 1.27 1.27)) (justify left))
     )
-    (property "Value" "100K" (id 1) (at 274.32 200.6599 0)
+    (property "Value" "1.5k" (id 1) (at 274.32 200.6599 0)
       (effects (font (size 1.27 1.27)) (justify left))
     )
@@
       (effects (font (size 1.27 1.27)) (justify left))
     )
-    (property "Value" "3K" (id 1) (at 83.82 116.8401 0)
+    (property "Value" "3.3K" (id 1) (at 83.82 116.8401 0)
       (effects (font (size 1.27 1.27)) (justify left))
     )
@@
     )
     (path "/0ac437c1-68f4-46a8-b149-23e59a83aa60"
-      (reference "C5") (unit 1) (value "33n") (footprint "Capacitor_SMD:C_0805_2012Metric")
+      (reference "C5") (unit 1) (value "330n") (footprint "Capacitor_SMD:C_0805_2012Metric")
     )
     (path "/27f7a360-b292-433a-a38b-e2b86826bc8e"
-      (reference "C6") (unit 1) (value "1n") (footprint "Capacitor_SMD:C_0805_2012Metric")
+      (reference "C6") (unit 1) (value "100n") (footprint "Capacitor_SMD:C_0805_2012Metric")
     )
     (path "/52bc58b8-747d-47aa-b4e0-750d9a663967"
@@
     )
     (path "/5d9af7fa-bed5-49c4-8cfc-eff4ea4151c5"
-      (reference "R1") (unit 1) (value "1K") (footprint "Resistor_SMD:R_0805_2012Metric")
+      (reference "R1") (unit 1) (value "180") (footprint "Resistor_SMD:R_0805_2012Metric")
     )
     (path "/a8657f7b-3339-4639-b150-22dc571735b8"
-      (reference "R2") (unit 1) (value "1K") (footprint "Resistor_SMD:R_0805_2012Metric")
+      (reference "R2") (unit 1) (value "180") (footprint "Resistor_SMD:R_0805_2012Metric")
     )
     (path "/2ec439f9-b91b-4644-b49d-c78c317ac589"
@@
     )
     (path "/f8477a63-bfb1-41f3-92e0-ecca5efe0b9b"
-      (reference "R8") (unit 1) (value "3K") (footprint "Resistor_SMD:R_0805_2012Metric")
+      (reference "R8") (unit 1) (value "3.3K") (footprint "Resistor_SMD:R_0805_2012Metric")
     )
     (path "/c88c5ded-10ba-40cd-8583-a8be601010f3"
@@
     )
     (path "/6153ef39-742a-491a-9781-05738f51ada2"
-      (reference "R14") (unit 1) (value "150K") (footprint "Resistor_SMD:R_0805_2012Metric")
+      (reference "R14") (unit 1) (value "1.5K") (footprint "Resistor_SMD:R_0805_2012Metric")
     )
     (path "/27b2a2a3-c147-466a-89ad-2ddb056c9338"
-      (reference "R15") (unit 1) (value "75K") (footprint "Resistor_SMD:R_0805_2012Metric")
+      (reference "R15") (unit 1) (value "750") (footprint "Resistor_SMD:R_0805_2012Metric")
     )
     (path "/65fd411b-e96a-4ede-92b9-42f55ae4daa3"
-      (reference "R16") (unit 1) (value "430K") (footprint "Resistor_SMD:R_0805_2012Metric")
+      (reference "R16") (unit 1) (value "4.3K") (footprint "Resistor_SMD:R_0805_2012Metric")
     )
     (path "/d6ce1335-c02c-4dab-be32-1a6974cc508b"
-      (reference "R17") (unit 1) (value "100K") (footprint "Resistor_SMD:R_0805_2012Metric")
+      (reference "R17") (unit 1) (value "1K") (footprint "Resistor_SMD:R_0805_2012Metric")
     )
     (path "/56940fd4-116e-4cb8-8651-2837cb5de83d"
-      (reference "R18") (unit 1) (value "110K") (footprint "Resistor_SMD:R_0805_2012Metric")
+      (reference "R18") (unit 1) (value "2k") (footprint "Resistor_SMD:R_0805_2012Metric")
     )
     (path "/8fd0fad3-a923-4a26-b5dd-366167f93eb1"
@@
     )
     (path "/e7a60f46-281c-4b22-8018-9769cacab751"
-      (reference "R21") (unit 1) (value "100K") (footprint "Resistor_SMD:R_0805_2012Metric")
+      (reference "R21") (unit 1) (value "1.5k") (footprint "Resistor_SMD:R_0805_2012Metric")
     )
     (path "/9ca806e0-98da-48c6-82cf-c01e5ea3b5dc"
@@
     )
     (path "/2474b851-43a4-439b-8b80-2f73777d1ba3"
-      (reference "R30") (unit 1) (value "110K") (footprint "Resistor_SMD:R_0805_2012Metric")
+      (reference "R30") (unit 1) (value "2K") (footprint "Resistor_SMD:R_0805_2012Metric")
     )
     (path "/e6f25c3a-9976-43cf-bb39-47facf09bf0c"
-      (reference "R31") (unit 1) (value "100K") (footprint "Resistor_SMD:R_0805_2012Metric")
+      (reference "R31") (unit 1) (value "1.5K") (footprint "Resistor_SMD:R_0805_2012Metric")
     )
     (path "/496e6ec2-b5b1-4e8e-9852-81bce44b2c2b"
@@
     )
     (path "/e6605161-e91a-4b46-b3d5-6601b9d1fb1e"
-      (reference "R41") (unit 1) (value "2K") (footprint "Resistor_SMD:R_0805_2012Metric")
+      (reference "R41") (unit 1) (value "350") (footprint "Resistor_SMD:R_0805_2012Metric")
     )
     (path "/922910b6-bf60-4061-8394-2b6464adaed8"

Commit message: fix board
Parts:
- R1, R2: value 180 -> 300
- R22, R23: value 2K -> 1K
- R4, R5: value 47k -> 1k
- R41: value 350 -> 680
- R48, R52: value 90k -> 1.5k
- R8: value 3.3K -> 2.4K
Changed lines of the file:
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@@
     (in_bom yes) (on_board yes) (fields_autoplaced)
     (property "Reference" "R48" (id 0) (at 246.38 45.72 90))
-    (property "Value" "90k" (id 1) (at 246.38 48.26 90))
+    (property "Value" "1.5k" (id 1) (at 246.38 48.26 90))
     (property "Footprint" "Resistor_SMD:R_0805_2012Metric" (id 2) (at 246.38 53.848 90)
       (effects (font (size 1.27 1.27)) hide)
@@
     (in_bom yes) (on_board yes) (fields_autoplaced)
     (property "Reference" "R1" (id 0) (at 220.98 45.72 90))
-    (property "Value" "180" (id 1) (at 220.98 48.26 90))
+    (property "Value" "300" (id 1) (at 220.98 48.26 90))
     (property "Footprint" "Resistor_SMD:R_0805_2012Metric" (id 2) (at 220.98 53.848 90)
       (effects (font (size 1.27 1.27)) hide)
@@
       (effects (font (size 1.27 1.27)) (justify left))
     )
-    (property "Value" "2K" (id 1) (at 138.43 95.2501 0)
+    (property "Value" "1K" (id 1) (at 138.43 95.2501 0)
       (effects (font (size 1.27 1.27)) (justify left))
     )
@@
     (in_bom yes) (on_board yes) (fields_autoplaced)
     (property "Reference" "R4" (id 0) (at 256.54 45.72 90))
-    (property "Value" "47k" (id 1) (at 256.54 48.26 90))
+    (property "Value" "1k" (id 1) (at 256.54 48.26 90))
     (property "Footprint" "Resistor_SMD:R_0805_2012Metric" (id 2) (at 256.54 53.848 90)
       (effects (font (size 1.27 1.27)) hide)
@@
     (in_bom yes) (on_board yes) (fields_autoplaced)
     (property "Reference" "R5" (id 0) (at 256.54 62.23 90))
-    (property "Value" "47k" (id 1) (at 256.54 64.77 90))
+    (property "Value" "1k" (id 1) (at 256.54 64.77 90))
     (property "Footprint" "Resistor_SMD:R_0805_2012Metric" (id 2) (at 256.54 70.358 90)
       (effects (font (size 1.27 1.27)) hide)
@@
       (effects (font (size 1.27 1.27)) (justify left))
     )
-    (property "Value" "2K" (id 1) (at 143.51 90.1699 0)
+    (property "Value" "1K" (id 1) (at 143.51 90.1699 0)
       (effects (font (size 1.27 1.27)) (justify left))
     )
@@
     (in_bom yes) (on_board yes) (fields_autoplaced)
     (property "Reference" "R2" (id 0) (at 220.98 62.23 90))
-    (property "Value" "180" (id 1) (at 220.98 64.77 90))
+    (property "Value" "300" (id 1) (at 220.98 64.77 90))
     (property "Footprint" "Resistor_SMD:R_0805_2012Metric" (id 2) (at 220.98 70.358 90)
       (effects (font (size 1.27 1.27)) hide)
@@
     (in_bom yes) (on_board yes) (fields_autoplaced)
     (property "Reference" "R52" (id 0) (at 246.38 62.23 90))
-    (property "Value" "90k" (id 1) (at 246.38 64.77 90))
+    (property "Value" "1.5k" (id 1) (at 246.38 64.77 90))
     (property "Footprint" "Resistor_SMD:R_0805_2012Metric" (id 2) (at 246.38 70.358 90)
       (effects (font (size 1.27 1.27)) hide)
@@
       (effects (font (size 1.27 1.27)) (justify left))
     )
-    (property "Value" "350" (id 1) (at 245.1101 118.11 0)
+    (property "Value" "680" (id 1) (at 245.1101 118.11 0)
       (effects (font (size 1.27 1.27)) (justify left))
     )
@@
       (effects (font (size 1.27 1.27)) (justify left))
     )
-    (property "Value" "3.3K" (id 1) (at 83.82 116.8401 0)
+    (property "Value" "2.4K" (id 1) (at 83.82 116.8401 0)
       (effects (font (size 1.27 1.27)) (justify left))
     )
@@
     )
     (path "/5d9af7fa-bed5-49c4-8cfc-eff4ea4151c5"
-      (reference "R1") (unit 1) (value "180") (footprint "Resistor_SMD:R_0805_2012Metric")
+      (reference "R1") (unit 1) (value "300") (footprint "Resistor_SMD:R_0805_2012Metric")
     )
     (path "/a8657f7b-3339-4639-b150-22dc571735b8"
-      (reference "R2") (unit 1) (value "180") (footprint "Resistor_SMD:R_0805_2012Metric")
+      (reference "R2") (unit 1) (value "300") (footprint "Resistor_SMD:R_0805_2012Metric")
     )
     (path "/2ec439f9-b91b-4644-b49d-c78c317ac589"
@@
     )
     (path "/68feafb5-7641-44b7-8eff-cc6981d24916"
-      (reference "R4") (unit 1) (value "47k") (footprint "Resistor_SMD:R_0805_2012Metric")
+      (reference "R4") (unit 1) (value "1k") (footprint "Resistor_SMD:R_0805_2012Metric")
     )
     (path "/8eff6cc6-648f-47e0-84e1-7d46250ee8cd"
-      (reference "R5") (unit 1) (value "47k") (footprint "Resistor_SMD:R_0805_2012Metric")
+      (reference "R5") (unit 1) (value "1k") (footprint "Resistor_SMD:R_0805_2012Metric")
     )
     (path "/24d3d6cc-3184-4dfc-bbb9-a05da1366057"
@@
     )
     (path "/f8477a63-bfb1-41f3-92e0-ecca5efe0b9b"
-      (reference "R8") (unit 1) (value "3.3K") (footprint "Resistor_SMD:R_0805_2012Metric")
+      (reference "R8") (unit 1) (value "2.4K") (footprint "Resistor_SMD:R_0805_2012Metric")
     )
     (path "/c88c5ded-10ba-40cd-8583-a8be601010f3"
@@
     )
     (path "/9ca806e0-98da-48c6-82cf-c01e5ea3b5dc"
-      (reference "R22") (unit 1) (value "2K") (footprint "Resistor_SMD:R_0805_2012Metric")
+      (reference "R22") (unit 1) (value "1K") (footprint "Resistor_SMD:R_0805_2012Metric")
     )
     (path "/68c4bfcd-8754-470c-b082-f86ccabca3df"
-      (reference "R23") (unit 1) (value "2K") (footprint "Resistor_SMD:R_0805_2012Metric")
+      (reference "R23") (unit 1) (value "1K") (footprint "Resistor_SMD:R_0805_2012Metric")
     )
     (path "/7d38fa5a-92ca-4d23-89f0-971df42386b1"
@@
     )
     (path "/e6605161-e91a-4b46-b3d5-6601b9d1fb1e"
-      (reference "R41") (unit 1) (value "350") (footprint "Resistor_SMD:R_0805_2012Metric")
+      (reference "R41") (unit 1) (value "680") (footprint "Resistor_SMD:R_0805_2012Metric")
     )
     (path "/922910b6-bf60-4061-8394-2b6464adaed8"
@@
     )
     (path "/51841b42-4827-42ac-9c06-c23d85bf953d"
-      (reference "R48") (unit 1) (value "90k") (footprint "Resistor_SMD:R_0805_2012Metric")
+      (reference "R48") (unit 1) (value "1.5k") (footprint "Resistor_SMD:R_0805_2012Metric")
     )
     (path "/67d0089f-a566-4ef5-b7cb-744e353a5220"
@@
     )
     (path "/c2430710-e764-4052-8fe3-28953a1b3099"
-      (reference "R52") (unit 1) (value "90k") (footprint "Resistor_SMD:R_0805_2012Metric")
+      (reference "R52") (unit 1) (value "1.5k") (footprint "Resistor_SMD:R_0805_2012Metric")
     )
     (path "/4898db39-c11d-4ee7-b12f-32821e63ef63"
